File: Comms_board.sch (KiCad schematic (older format))
At the start: 0 parts

Commit message: first test
Other:
- note added: "test text"
Changed lines of the file:
@@
 LIBS:contrib
 LIBS:valves
+LIBS:Comms_board-cache
 EELAYER 25 0
 EELAYER END
@@
 Comment4 ""
 $EndDescr
-Text Label 4350 1200 0    60   ~ 0
-test
+Text Notes 3650 2450 0    60   ~ 0
+test text
 $EndSCHEMATC

Commit message: removed test
Other:
- note removed: "test text"
Changed lines of the file:
@@
 Comment4 ""
 $EndDescr
-Text Notes 3650 2450 0    60   ~ 0
-test text
 $EndSCHEMATC

Commit message: converted .bxl file into KiCAD schematic/footprint library
Parts:
- added U?: CC1120RHB, RHB0032E, symbol CC1120RHB
Connections:
- new net Earth: U?.33 (GND)
Changed lines of the file:
@@
 LIBS:contrib
 LIBS:valves
+LIBS:MSSG_CC1120
 LIBS:Comms_board-cache
 EELAYER 25 0
@@
 Comment4 ""
 $EndDescr
+$Comp
+L CC1120RHB U?
+U 1 1 5942115C
+P 5250 3700
+F 0 "U?" H 5250 3800 60  0000 C CNN
+F 1 "CC1120RHB" H 5250 3700 60  0000 C CNN
+F 2 "RHB0032E" H 5250 3640 60  0001 C CNN
+F 3 "" H 5250 3700 60  0000 C CNN
+	1    5250 3700
+	1    0    0    -1
+$EndComp
+$Comp
+L Earth #PWR?
+U 1 1 5942167F
+P 6550 5250
+F 0 "#PWR?" H 6550 5000 50  0001 C CNN
+F 1 "Earth" H 6550 5100 50  0001 C CNN
+F 2 "" H 6550 5250 50  0001 C CNN
+F 3 "" H 6550 5250 50  0001 C CNN
+	1    6550 5250
+	1    0    0    -1
+$EndComp
+Wire Wire Line
+	6350 5100 6550 5100
+Wire Wire Line
+	6550 5100 6550 5250
 $EndSCHEMATC
